File: proto2/power.sch (KiCad schematic (older format))
At the start: 2 parts, among them U13 AP1117-50, U14 JTD1548S15

Commit message: Added note for current draw of SBCs.
Other:
- note added: "Raspberry Pi draws 1.3A and recomends 2.5A @ 5V.\nBeagleBone draws 1.2A and recomends at least 2A."
Changed lines of the file:
@@
 	1    0    0    -1
 $EndComp
+Text Notes 2550 1000 0    50   ~ 0
+Raspberry Pi draws 1.3A and recomends 2.5A @ 5V.\nBeagleBone draws 1.2A and recomends at least 2A.
 $EndSCHEMATC
