File: proto2/outputs.kicad_sch (KiCad schematic)
At the start: 84 parts, among them Q1 2N7002, Q10 2N7002, Q11 2N7002, Q12 2N7002, Q13 2N7002, Q14 2N7002, Q2 2N7002, Q3 2N7002, Q4 2N7002, Q5 2N7002, Q6 2N7002, Q7 2N7002, Q8 2N7002, Q9 2N7002, U1 AQY282SX, U10 AQY282SX, U11 AQY282SX, U12 AQY282SX, U13 AQY282SX, U14 AQY282SX, U2 AQY282SX, U3 AQY282SX, U4 AQY282SX, U5 AQY282SX, U6 AQY282SX, U7 AQY282SX, U8 AQY282SX, U9 AQY282SX

Commit message: Updated PTC sizes so they will not trip with typical current draw.
Parts:
- F1, F10, F11, F12, F13, F14, F2, F3, F4, F5, F6, F7, F8, F9: LCSC C70070 -> C70077
Changed lines of the file:
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@@
       (effects (font (size 1.27 1.27)) (justify left) hide)
     )
-    (property "Datasheet" "https://datasheet.lcsc.com/lcsc/1811031612_TECHFUSE-nSMD025-30V_C70070.pdf" (id 3) (at 78.74 25.4 0)
-      (effects (font (size 1.27 1.27)) hide)
-    )
-    (property "LCSC" "C70070" (id 4) (at 78.74 25.4 0)
+    (property "Datasheet" "https://datasheet.lcsc.com/lcsc/1809211126_TECHFUSE-nSMD050-33V_C70077.pdf" (id 3) (at 78.74 25.4 0)
+      (effects (font (size 1.27 1.27)) hide)
+    )
+    (property "LCSC" "C70077" (id 4) (at 78.74 25.4 0)
       (effects (font (size 1.27 1.27)) hide)
     )
@@
       (effects (font (size 1.27 1.27)) (justify left) hide)
     )
-    (property "Datasheet" "https://datasheet.lcsc.com/lcsc/1811031612_TECHFUSE-nSMD025-30V_C70070.pdf" (id 3) (at 76.2 59.69 0)
-      (effects (font (size 1.27 1.27)) hide)
-    )
-    (property "LCSC" "C70070" (id 4) (at 76.2 59.69 0)
+    (property "Datasheet" "https://datasheet.lcsc.com/lcsc/1809211126_TECHFUSE-nSMD050-33V_C70077.pdf" (id 3) (at 76.2 59.69 0)
+      (effects (font (size 1.27 1.27)) hide)
+    )
+    (property "LCSC" "C70077" (id 4) (at 76.2 59.69 0)
       (effects (font (size 1.27 1.27)) hide)
     )
@@
       (effects (font (size 1.27 1.27)) (justify left) hide)
     )
-    (property "Datasheet" "https://datasheet.lcsc.com/lcsc/1811031612_TECHFUSE-nSMD025-30V_C70070.pdf" (id 3) (at 77.47 92.71 0)
-      (effects (font (size 1.27 1.27)) hide)
-    )
-    (property "LCSC" "C70070" (id 4) (at 77.47 92.71 0)
+    (property "Datasheet" "https://datasheet.lcsc.com/lcsc/1809211126_TECHFUSE-nSMD050-33V_C70077.pdf" (id 3) (at 77.47 92.71 0)
+      (effects (font (size 1.27 1.27)) hide)
+    )
+    (property "LCSC" "C70077" (id 4) (at 77.47 92.71 0)
       (effects (font (size 1.27 1.27)) hide)
     )
@@
       (effects (font (size 1.27 1.27)) (justify left) hide)
     )
-    (property "Datasheet" "https://datasheet.lcsc.com/lcsc/1811031612_TECHFUSE-nSMD025-30V_C70070.pdf" (id 3) (at 78.74 125.73 0)
-      (effects (font (size 1.27 1.27)) hide)
-    )
-    (property "LCSC" "C70070" (id 4) (at 78.74 125.73 0)
+    (property "Datasheet" "https://datasheet.lcsc.com/lcsc/1809211126_TECHFUSE-nSMD050-33V_C70077.pdf" (id 3) (at 78.74 125.73 0)
+      (effects (font (size 1.27 1.27)) hide)
+    )
+    (property "LCSC" "C70077" (id 4) (at 78.74 125.73 0)
       (effects (font (size 1.27 1.27)) hide)
     )
@@
       (effects (font (size 1.27 1.27)) (justify left) hide)
     )
-    (property "Datasheet" "https://datasheet.lcsc.com/lcsc/1811031612_TECHFUSE-nSMD025-30V_C70070.pdf" (id 3) (at 161.29 25.4 0)
-      (effects (font (size 1.27 1.27)) hide)
-    )
-    (property "LCSC" "C70070" (id 4) (at 161.29 25.4 0)
+    (property "Datasheet" "https://datasheet.lcsc.com/lcsc/1809211126_TECHFUSE-nSMD050-33V_C70077.pdf" (id 3) (at 161.29 25.4 0)
+      (effects (font (size 1.27 1.27)) hide)
+    )
+    (property "LCSC" "C70077" (id 4) (at 161.29 25.4 0)
       (effects (font (size 1.27 1.27)) hide)
     )
@@
       (effects (font (size 1.27 1.27)) (justify left) hide)
     )
-    (property "Datasheet" "https://datasheet.lcsc.com/lcsc/1811031612_TECHFUSE-nSMD025-30V_C70070.pdf" (id 3) (at 160.02 59.69 0)
-      (effects (font (size 1.27 1.27)) hide)
-    )
-    (property "LCSC" "C70070" (id 4) (at 160.02 59.69 0)
+    (property "Datasheet" "https://datasheet.lcsc.com/lcsc/1809211126_TECHFUSE-nSMD050-33V_C70077.pdf" (id 3) (at 160.02 59.69 0)
+      (effects (font (size 1.27 1.27)) hide)
+    )
+    (property "LCSC" "C70077" (id 4) (at 160.02 59.69 0)
       (effects (font (size 1.27 1.27)) hide)
     )
@@
       (effects (font (size 1.27 1.27)) (justify left) hide)
     )
-    (property "Datasheet" "https://datasheet.lcsc.com/lcsc/1811031612_TECHFUSE-nSMD025-30V_C70070.pdf" (id 3) (at 161.29 92.71 0)
-      (effects (font (size 1.27 1.27)) hide)
-    )
-    (property "LCSC" "C70070" (id 4) (at 161.29 92.71 0)
+    (property "Datasheet" "https://datasheet.lcsc.com/lcsc/1809211126_TECHFUSE-nSMD050-33V_C70077.pdf" (id 3) (at 161.29 92.71 0)
+      (effects (font (size 1.27 1.27)) hide)
+    )
+    (property "LCSC" "C70077" (id 4) (at 161.29 92.71 0)
       (effects (font (size 1.27 1.27)) hide)
     )
@@
       (effects (font (size 1.27 1.27)) (justify left) hide)
     )
-    (property "Datasheet" "https://datasheet.lcsc.com/lcsc/1811031612_TECHFUSE-nSMD025-30V_C70070.pdf" (id 3) (at 158.75 125.73 0)
-      (effects (font (size 1.27 1.27)) hide)
-    )
-    (property "LCSC" "C70070" (id 4) (at 158.75 125.73 0)
+    (property "Datasheet" "https://datasheet.lcsc.com/lcsc/1809211126_TECHFUSE-nSMD050-33V_C70077.pdf" (id 3) (at 158.75 125.73 0)
+      (effects (font (size 1.27 1.27)) hide)
+    )
+    (property "LCSC" "C70077" (id 4) (at 158.75 125.73 0)
       (effects (font (size 1.27 1.27)) hide)
     )
@@
       (effects (font (size 1.27 1.27)) (justify left) hide)
     )
-    (property "Datasheet" "https://datasheet.lcsc.com/lcsc/1811031612_TECHFUSE-nSMD025-30V_C70070.pdf" (id 3) (at 246.38 25.4 0)
-      (effects (font (size 1.27 1.27)) hide)
-    )
-    (property "LCSC" "C70070" (id 4) (at 246.38 25.4 0)
+    (property "Datasheet" "https://datasheet.lcsc.com/lcsc/1809211126_TECHFUSE-nSMD050-33V_C70077.pdf" (id 3) (at 246.38 25.4 0)
+      (effects (font (size 1.27 1.27)) hide)
+    )
+    (property "LCSC" "C70077" (id 4) (at 246.38 25.4 0)
       (effects (font (size 1.27 1.27)) hide)
     )
@@
       (effects (font (size 1.27 1.27)) (justify left) hide)
     )
-    (property "Datasheet" "https://datasheet.lcsc.com/lcsc/1811031612_TECHFUSE-nSMD025-30V_C70070.pdf" (id 3) (at 243.84 59.69 0)
-      (effects (font (size 1.27 1.27)) hide)
-    )
-    (property "LCSC" "C70070" (id 4) (at 243.84 59.69 0)
+    (property "Datasheet" "https://datasheet.lcsc.com/lcsc/1809211126_TECHFUSE-nSMD050-33V_C70077.pdf" (id 3) (at 243.84 59.69 0)
+      (effects (font (size 1.27 1.27)) hide)
+    )
+    (property "LCSC" "C70077" (id 4) (at 243.84 59.69 0)
       (effects (font (size 1.27 1.27)) hide)
     )
@@
       (effects (font (size 1.27 1.27)) (justify left) hide)
     )
-    (property "Datasheet" "https://datasheet.lcsc.com/lcsc/1811031612_TECHFUSE-nSMD025-30V_C70070.pdf" (id 3) (at 245.11 92.71 0)
-      (effects (font (size 1.27 1.27)) hide)
-    )
-    (property "LCSC" "C70070" (id 4) (at 245.11 92.71 0)
+    (property "Datasheet" "https://datasheet.lcsc.com/lcsc/1809211126_TECHFUSE-nSMD050-33V_C70077.pdf" (id 3) (at 245.11 92.71 0)
+      (effects (font (size 1.27 1.27)) hide)
+    )
+    (property "LCSC" "C70077" (id 4) (at 245.11 92.71 0)
       (effects (font (size 1.27 1.27)) hide)
     )
@@
       (effects (font (size 1.27 1.27)) (justify left) hide)
     )
-    (property "Datasheet" "https://datasheet.lcsc.com/lcsc/1811031612_TECHFUSE-nSMD025-30V_C70070.pdf" (id 3) (at 246.38 125.73 0)
-      (effects (font (size 1.27 1.27)) hide)
-    )
-    (property "LCSC" "C70070" (id 4) (at 246.38 125.73 0)
+    (property "Datasheet" "https://datasheet.lcsc.com/lcsc/1809211126_TECHFUSE-nSMD050-33V_C70077.pdf" (id 3) (at 246.38 125.73 0)
+      (effects (font (size 1.27 1.27)) hide)
+    )
+    (property "LCSC" "C70077" (id 4) (at 246.38 125.73 0)
       (effects (font (size 1.27 1.27)) hide)
     )
@@
       (effects (font (size 1.27 1.27)) (justify left) hide)
     )
-    (property "Datasheet" "https://datasheet.lcsc.com/lcsc/1811031612_TECHFUSE-nSMD025-30V_C70070.pdf" (id 3) (at 78.74 160.02 0)
-      (effects (font (size 1.27 1.27)) hide)
-    )
-    (property "LCSC" "C70070" (id 4) (at 78.74 160.02 0)
+    (property "Datasheet" "https://datasheet.lcsc.com/lcsc/1809211126_TECHFUSE-nSMD050-33V_C70077.pdf" (id 3) (at 78.74 160.02 0)
+      (effects (font (size 1.27 1.27)) hide)
+    )
+    (property "LCSC" "C70077" (id 4) (at 78.74 160.02 0)
       (effects (font (size 1.27 1.27)) hide)
     )
@@
       (effects (font (size 1.27 1.27)) (justify left) hide)
     )
-    (property "Datasheet" "https://datasheet.lcsc.com/lcsc/1811031612_TECHFUSE-nSMD025-30V_C70070.pdf" (id 3) (at 161.29 160.02 0)
-      (effects (font (size 1.27 1.27)) hide)
-    )
-    (property "LCSC" "C70070" (id 4) (at 161.29 160.02 0)
-      (effects (font (size 1.27 1.27)) hide)
-    )
+    (property "Datasheet" "https://datasheet.lcsc.com/lcsc/1809211126_TECHFUSE-nSMD050-33V_C70077.pdf" (id 3) (at 161.29 160.02 0)
+      (effects (font (size 1.27 1.27)) hide)
+    )
+    (property "LCSC" "C70077" (id 4) (at 161.29 160.02 0)
+      (effects (font (size 1.27 1.27)) hide)
+    )
