File: proto2/outputs.kicad_sch (KiCad schematic)
At the start: 84 parts, among them Q1 2N7002, Q10 2N7002, Q11 2N7002, Q12 2N7002, Q13 2N7002, Q14 2N7002, Q2 2N7002, Q3 2N7002, Q4 2N7002, Q5 2N7002, Q6 2N7002, Q7 2N7002, Q8 2N7002, Q9 2N7002, U1 TLP240A, U10 TLP240A, U11 TLP240A, U12 TLP240A, U13 TLP240A, U14 TLP240A, U2 TLP240A, U3 TLP240A, U4 TLP240A, U5 TLP240A, U6 TLP240A, U7 TLP240A, U8 TLP240A, U9 TLP240A

Commit message: Changed paper size and some text on the titleblocks
Other:
- company: Langhe Greenhaus -> Langhe
- title: Greenhouse 2.0 IO Board -> IO Board
Changed lines of the file:
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@@
   (paper "USLetter")
   (title_block
-    (title "Greenhouse 2.0 IO Board")
+    (title "IO Board")
     (date "2022-09-13")
     (rev "0.3.2")
-    (company "Langhe Greenhaus")
-    (comment 1 "Langhe Part Number: 240000")
+    (company "Langhe")
   )
   (junction (at 36.83 100.33) (diameter 0) (color 0 0 0 0)
