File: proto2/terminals2.kicad_sch (KiCad schematic)
At the start: 161 parts, among them J2 Output, J3 Output, J4 Output, J5 Output, J6 Output, J7 Output, J8 Output

Commit message: Laying out board. in-process commit.
Changed lines of the file:
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@@
   (title_block
     (title "Greenhouse 2.0 IO Board")
-    (date "2022-02-22")
+    (date "2022-02-24")
     (rev "0.2.0")
     (company "Langhe Greenhaus")
@@
     (stroke (width 0) (type default) (color 0 0 0 0))
   )
-  (wire (pts (xy 21.59 39.37) (xy 21.59 34.29))
-    (stroke (width 0) (type default) (color 0 0 0 0))
-  )
   (wire (pts (xy 45.72 96.52) (xy 45.72 105.41))
     (stroke (width 0) (type default) (color 0 0 0 0))
   )
-  (wire (pts (xy 21.59 34.29) (xy 17.78 34.29))
-    (stroke (width 0) (type default) (color 0 0 0 0))
-  )
   (wire (pts (xy 139.7 176.53) (xy 143.51 176.53))
     (stroke (width 0) (type default) (color 0 0 0 0))
@@
     (stroke (width 0) (type default) (color 0 0 0 0))
   )
-  (label "PWRGND" (at 17.78 34.29 0)
-    (effects (font (size 1.27 1.27)) (justify left bottom))
-  )
   (global_label "DQ1_2" (shape input) (at 30.48 29.21 180) (fields_autoplaced)
     (effects (font (size 1.27 1.27)) (justify right))
@@
     (pin "2")
   )
-  (symbol (lib_id "Power_BCR:PWRGND") (at 21.59 39.37 0) (mirror y) (unit 1)
-    (in_bom yes) (on_board yes)
-    (property "Reference" "#PWR0246" (id 0) (at 21.59 45.72 0)
-      (effects (font (size 1.27 1.27)) hide)
-    )
-    (property "Value" "PWRGND" (id 1) (at 21.59 43.18 0)
-      (effects (font (size 1.27 1.27)) hide)
-    )
-    (property "Footprint" "" (id 2) (at 21.59 39.37 0)
-      (effects (font (size 1.27 1.27)) hide)
-    )
-    (property "Datasheet" "~" (id 3) (at 21.59 39.37 0)
-      (effects (font (size 1.27 1.27)) hide)
-    )
-    (pin "1")
-  )
   (symbol (lib_id "Connector_Generic:Conn_01x04") (at 148.59 171.45 0) (unit 1)

Commit message: Final layout for 0.2.0 and various BOM and minor schematic updates.
Parts:
- J2, J3, J4, J5, J6, J7, J8: MPN (none) -> DNP
Changed lines of the file:
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@@
+      (effects (font (size 1.27 1.27)) hide)
+    )
+    (property "MPN" "DNP" (id 4) (at 148.59 26.67 0)
       (effects (font (size 1.27 1.27)) hide)
     )
@@
       (effects (font (size 1.27 1.27)) hide)
     )
+    (property "MPN" "DNP" (id 4) (at 148.59 50.8 0)
+      (effects (font (size 1.27 1.27)) hide)
+    )
     (pin "1")
     (pin "2")
@@
       (effects (font (size 1.27 1.27)) hide)
     )
+    (property "MPN" "DNP" (id 4) (at 148.59 74.93 0)
+      (effects (font (size 1.27 1.27)) hide)
+    )
     (pin "1")
     (pin "2")
@@
       (effects (font (size 1.27 1.27)) hide)
     )
+    (property "MPN" "DNP" (id 4) (at 148.59 99.06 0)
+      (effects (font (size 1.27 1.27)) hide)
+    )
     (pin "1")
     (pin "2")
@@
       (effects (font (size 1.27 1.27)) hide)
     )
+    (property "MPN" "DNP" (id 4) (at 148.59 123.19 0)
+      (effects (font (size 1.27 1.27)) hide)
+    )
     (pin "1")
     (pin "2")
@@
       (effects (font (size 1.27 1.27)) hide)
     )
+    (property "MPN" "DNP" (id 4) (at 148.59 147.32 0)
+      (effects (font (size 1.27 1.27)) hide)
+    )
     (pin "1")
     (pin "2")
@@
       (effects (font (size 1.27 1.27)) hide)
     )
+    (property "MPN" "DNP" (id 4) (at 148.59 171.45 0)
+      (effects (font (size 1.27 1.27)) hide)
+    )
