File: proto2/terminals2.kicad_sch (KiCad schematic)
At the start: 161 parts, among them J2 Output, J3 Output, J4 Output, J5 Output, J6 Output, J7 Output, J8 Output

Commit message: Changed paper size and some text on the titleblocks
Other:
- company: Langhe Greenhaus -> Langhe
- title: Greenhouse 2.0 IO Board -> IO Board
Changed lines of the file:
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@@
   (paper "USLetter")
   (title_block
-    (title "Greenhouse 2.0 IO Board")
+    (title "IO Board")
     (date "2022-09-13")
     (rev "0.3.2")
-    (company "Langhe Greenhaus")
-    (comment 1 "Langhe Part Number: 240000")
+    (company "Langhe")
   )
   (junction (at 115.57 55.88) (diameter 0) (color 0 0 0 0)
