File: proto2/inputs.kicad_sch (KiCad schematic)
At the start: 14 parts, among them U19 EL817S1, U20 EL817S1, U21 EL817S1, U22 EL817S1

Commit message: Changed paper size and some text on the titleblocks
Other:
- company: Langhe Greenhaus -> Langhe
- title: Greenhouse 2.0 IO Board -> IO Board
Changed lines of the file:
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@@
 (kicad_sch (version 20230121) (generator eeschema)
-  (paper "A4")
+  (paper "USLetter")
   (title_block
-    (title "Greenhouse 2.0 IO Board")
+    (title "IO Board")
     (date "2022-09-13")
     (rev "0.3.2")
-    (company "Langhe Greenhaus")
-    (comment 1 "Langhe Part Number: 240000")
+    (company "Langhe")
   )
   (junction (at 114.3 124.46) (diameter 0) (color 0 0 0 0)
