File: proto2/proto2.kicad_sch (KiCad schematic)
At the start: 15 parts, among them J13 Daughter Card, J17 Conn_01x06, SW1 SW_DIP_x04, U16 ADS1015IDGS

Commit message: Changed paper size and some text on the titleblocks
Other:
- company: Langhe Greenhaus -> Langhe
- title: Greenhouse 2.0 IO Board -> IO Board
Changed lines of the file:
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@@
   (paper "USLetter")
   (title_block
-    (title "Greenhouse 2.0 IO Board")
+    (title "IO Board")
     (date "2022-09-13")
     (rev "0.3.2")
-    (company "Langhe Greenhaus")
-    (comment 1 "Langhe Part Number: 240000")
+    (company "Langhe")
   )
   (junction (at 217.17 152.4) (diameter 0) (color 0 0 0 0)
