File: proto2/terminals.kicad_sch (KiCad schematic)
At the start: 75 parts, among them J1 Main Power, J10 Device, J11 Device, J12 Device, J9 Device

Commit message: Changed paper size and some text on the titleblocks
Other:
- company: Langhe Greenhaus -> Langhe
- title: Greenhouse 2.0 IO Board -> IO Board
Changed lines of the file:
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@@
   (paper "USLetter")
   (title_block
-    (title "Greenhouse 2.0 IO Board")
+    (title "IO Board")
     (date "2022-09-13")
     (rev "0.3.2")
-    (company "Langhe Greenhaus")
-    (comment 1 "Langhe Part Number: 240000")
+    (company "Langhe")
   )
   (junction (at 58.42 53.34) (diameter 0) (color 0 0 0 0)
